Commit message: First implementation of the optimization problem to find a suitable pose of the base. This first version is based on the alignment of the x-axis of the desired pose with the x-axis of the reference frame of the ellipsoid

File: reach_space_modeling/generate_pointcloud/model/mobile_wx250s.urdf (robot description, URDF)
Before this commit: robot mobile_wx250s, 15 links, 14 joints
Links:
- link locobot/ar_tag_link: geometry collision mesh filename=/home/rosario/Base-Pose-Optimization-for-Mobile-Robots/reac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 scale=0.001 0.001 0.001; visual mesh filename=/home/rosario/Base-Pose-Optimization-for-Mobile-Robots/reac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 scale=0.001 0.001 0.001
- link locobot/arm_base_link: geometry collision mesh filename=/home/rosario/Base-Pose-Optimization-for-Mobile-Robots/reac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 scale=0.001 0.001 0.001; visual mesh filename=/home/rosario/Base-Pose-Optimization-for-Mobile-Robots/reac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 scale=0.001 0.001 0.001
- link locobot/gripper_bar_link: geometry collision mesh filename=/home/rosario/Base-Pose-Optimization-for-Mobile-Robots/reac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 scale=0.001 0.001 0.001; visual mesh filename=/home/rosario/Base-Pose-Optimization-for-Mobile-Robots/reac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 scale=0.001 0.001 0.001
- link locobot/gripper_link: geometry collision mesh filename=/home/rosario/Base-Pose-Optimization-for-Mobile-Robots/reac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 scale=0.001 0.001 0.001; visual mesh filename=/home/rosario/Base-Pose-Optimization-for-Mobile-Robots/reac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 scale=0.001 0.001 0.001
- link locobot/gripper_prop_link: geometry collision mesh filename=/home/rosario/Base-Pose-Optimization-for-Mobile-Robots/reac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 scale=0.001 0.001 0.001; visual mesh filename=/home/rosario/Base-Pose-Optimization-for-Mobile-Robots/reac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 scale=0.001 0.001 0.001
- link locobot/left_finger_link: geometry collision mesh filename=/home/rosario/Base-Pose-Optimization-for-Mobile-Robots/reac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 scale=0.001 0.001 0.001; visual mesh filename=/home/rosario/Base-Pose-Optimization-for-Mobile-Robots/reac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 scale=0.001 0.001 0.001
- link locobot/lower_forearm_link: geometry collision mesh filename=/home/rosario/Base-Pose-Optimization-for-Mobile-Robots/reac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 scale=0.001 0.001 0.001; visual mesh filename=/home/rosario/Base-Pose-Optimization-for-Mobile-Robots/reac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 scale=0.001 0.001 0.001
- link locobot/right_finger_link: geometry collision mesh filename=/home/rosario/Base-Pose-Optimization-for-Mobile-Robots/reac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 scale=0.001 0.001 0.001; visual mesh filename=/home/rosario/Base-Pose-Optimization-for-Mobile-Robots/reac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 scale=0.001 0.001 0.001
- link locobot/shoulder_link: geometry collision mesh filename=/home/rosario/Base-Pose-Optimization-for-Mobile-Robots/reac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 scale=0.001 0.001 0.001; visual mesh filename=/home/rosario/Base-Pose-Optimization-for-Mobile-Robots/reac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 scale=0.001 0.001 0.001
- link locobot/upper_arm_link: geometry collision mesh filename=/home/rosario/Base-Pose-Optimization-for-Mobile-Robots/reac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 scale=0.001 0.001 0.001; visual mesh filename=/home/rosario/Base-Pose-Optimization-for-Mobile-Robots/reac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 scale=0.001 0.001 0.001
- link locobot/upper_forearm_link: geometry collision mesh filename=/home/rosario/Base-Pose-Optimization-for-Mobile-Robots/reac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 scale=0.001 0.001 0.001; visual mesh filename=/home/rosario/Base-Pose-Optimization-for-Mobile-Robots/reac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 scale=0.001 0.001 0.001
- link locobot/wrist_link: geometry collision mesh filename=/home/rosario/Base-Pose-Optimization-for-Mobile-Robots/reac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 scale=0.001 0.001 0.001; visual mesh filename=/home/rosario/Base-Pose-Optimization-for-Mobile-Robots/reac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 scale=0.001 0.001 0.001
